File: level_shifter.kicad_sch (KiCad schematic)
At the start: 5 parts

Commit message: Added USBC Connector to power page
Parts:
- gave numbers to parts that had none: 5
Changed lines of the file:
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@@
   (symbol (lib_id "arjun_symbols:CAP_CER_1u_25V_X5R_0603") (at 175.26 106.68 0) (unit 1)
     (in_bom yes) (on_board yes)
-    (property "Reference" "C?" (id 0) (at 178.308 107.696 0)
+    (property "Reference" "C8" (id 0) (at 178.308 107.696 0)
       (effects (font (size 1.27 1.27)) (justify left))
     )
@@
   (symbol (lib_id "arjun_symbols:CAP_CER_1u_25V_X5R_0603") (at 101.6 106.68 0) (unit 1)
     (in_bom yes) (on_board yes)
-    (property "Reference" "C?" (id 0) (at 104.648 107.696 0)
+    (property "Reference" "C5" (id 0) (at 104.648 107.696 0)
       (effects (font (size 1.27 1.27)) (justify left))
     )
@@
   (symbol (lib_id "power:GND") (at 119.38 99.06 0) (unit 1)
     (in_bom yes) (on_board yes)
-    (property "Reference" "#PWR?" (id 0) (at 119.38 105.41 0)
+    (property "Reference" "#PWR016" (id 0) (at 119.38 105.41 0)
       (effects (font (size 1.27 1.27)) hide)
     )
@@
   (symbol (lib_id "power:+3.3V") (at 101.6 101.6 0) (unit 1)
     (in_bom yes) (on_board yes)
-    (property "Reference" "#PWR?" (id 0) (at 101.6 105.41 0)
+    (property "Reference" "#PWR014" (id 0) (at 101.6 105.41 0)
       (effects (font (size 1.27 1.27)) hide)
     )
@@
   (symbol (lib_id "arjun_symbols:IC_LVL_MC14504BDTR2G") (at 121.92 78.74 0) (unit 1)
     (in_bom yes) (on_board yes)
-    (property "Reference" "U?" (id 0) (at 130.81 72.39 0)
+    (property "Reference" "U4" (id 0) (at 130.81 72.39 0)
       (effects (font (size 1.524 1.524)))
     )
@@
   (symbol (lib_id "power:GND") (at 101.6 119.38 0) (unit 1)
     (in_bom yes) (on_board yes)
-    (property "Reference" "#PWR?" (id 0) (at 101.6 125.73 0)
+    (property "Reference" "#PWR015" (id 0) (at 101.6 125.73 0)
       (effects (font (size 1.27 1.27)) hide)
     )
@@
   (symbol (lib_id "arjun_symbols:CAP_CER_0u1_50V_X7R_0603") (at 111.76 106.68 0) (unit 1)
     (in_bom yes) (on_board yes)
-    (property "Reference" "C?" (id 0) (at 114.808 107.696 0)
+    (property "Reference" "C6" (id 0) (at 114.808 107.696 0)
       (effects (font (size 1.27 1.27)) (justify left))
     )
@@
   (symbol (lib_id "power:+12V") (at 175.26 101.6 0) (unit 1)
     (in_bom yes) (on_board yes)
-    (property "Reference" "#PWR?" (id 0) (at 175.26 105.41 0)
+    (property "Reference" "#PWR017" (id 0) (at 175.26 105.41 0)
       (effects (font (size 1.27 1.27)) hide)
     )
@@
   (symbol (lib_id "arjun_symbols:CAP_CER_0u1_50V_X7R_0603") (at 165.1 106.68 0) (unit 1)
     (in_bom yes) (on_board yes)
-    (property "Reference" "C?" (id 0) (at 168.148 107.696 0)
+    (property "Reference" "C7" (id 0) (at 168.148 107.696 0)
       (effects (font (size 1.27 1.27)) (justify left))
     )
@@
   (symbol (lib_id "power:GND") (at 175.26 119.38 0) (unit 1)
     (in_bom yes) (on_board yes)
-    (property "Reference" "#PWR?" (id 0) (at 175.26 125.73 0)
-      (effects (font (size 1.27 1.27)) hide)
-    )
+    (property "Reference" "#PWR018" (id 0) (at 175.26 125.73 0)
+      (effects (font (size 1.27 1.27)) hide)
+    )
