File: power.kicad_sch (KiCad schematic)
At the start: 0 parts

Commit message: Added USBC Connector to power page
Parts:
- added C9: CAP_CER_4700p_250V_X7R_0805, Capacitor_SMD:C_0805_2012Metric, symbol arjun_symbols:CAP_CER_4700p_250V_X7R_0805
- added J1: CONN_USBC_RCPT_USB2.0_USB4085-GF-A, arjun_footprints:GCT_USB4085-GF-A_REVA4, symbol arjun_symbols:CONN_USBC_RCPT_USB2.0_USB4085-GF-A
- added R9: RES_0R_1/8W_0805, Resistor_SMD:R_0805_2012Metric, symbol arjun_symbols:RES_0R_1/8W_0805
- added R? (x2): RES_5K11_1P_1/10W_0603, Resistor_SMD:R_0603_1608Metric, symbol arjun_symbols:RES_5K11_1P_1/10W_0603
Connections:
- new net: J1.B5 (CC2), R?.1
- new net: J1.A5 (CC1), R?.1
- new net +5V: J1.A4 (VBUS), J1.A9 (VBUS), J1.B4 (VBUS), J1.B9 (VBUS)
- new net GND: C9.1, J1.A1 (GND), J1.A12 (GND), J1.B1 (GND), J1.B12 (GND), R9.2, R?.2, R?.2
- new net GNDPWR: C9.2, J1.S1 (SHIELD), J1.S2 (SHIELD), J1.S3 (SHIELD), J1.S4 (SHIELD), R9.1
- new net USB_D_N: J1.A7 (D-), J1.B7 (D-)
- new net USB_D_P: J1.A6 (D+), J1.B6 (D+)
- no-connect marks 0 -> 4
Other:
- note added: "DNP"
- note added: "Standard USB2.0 UFP Device"
