File: pcb/level_shifter.kicad_sch (KiCad schematic)
At the start: 5 parts, among them U4 IC_LVL_MC14504BDTR2G

Commit message: Added LSE crystal and started configuring MCU Pinout"
Parts:
- renumbered C5 to C13, C6 to C14, C7 to C15, C8 to C16
Changed lines of the file:
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@@
   (symbol (lib_id "arjun_symbols:CAP_CER_1u_25V_X5R_0603") (at 175.26 106.68 0) (unit 1)
     (in_bom yes) (on_board yes)
-    (property "Reference" "C8" (id 0) (at 178.308 107.696 0)
+    (property "Reference" "C16" (id 0) (at 178.308 107.696 0)
       (effects (font (size 1.27 1.27)) (justify left))
     )
@@
   (symbol (lib_id "arjun_symbols:CAP_CER_1u_25V_X5R_0603") (at 101.6 106.68 0) (unit 1)
     (in_bom yes) (on_board yes)
-    (property "Reference" "C5" (id 0) (at 104.648 107.696 0)
+    (property "Reference" "C13" (id 0) (at 104.648 107.696 0)
       (effects (font (size 1.27 1.27)) (justify left))
     )
@@
   (symbol (lib_id "power:GND") (at 119.38 99.06 0) (unit 1)
     (in_bom yes) (on_board yes)
-    (property "Reference" "#PWR016" (id 0) (at 119.38 105.41 0)
+    (property "Reference" "#PWR021" (id 0) (at 119.38 105.41 0)
       (effects (font (size 1.27 1.27)) hide)
     )
@@
   (symbol (lib_id "power:+3.3V") (at 101.6 101.6 0) (unit 1)
     (in_bom yes) (on_board yes)
-    (property "Reference" "#PWR014" (id 0) (at 101.6 105.41 0)
+    (property "Reference" "#PWR022" (id 0) (at 101.6 105.41 0)
       (effects (font (size 1.27 1.27)) hide)
     )
@@
   (symbol (lib_id "power:GND") (at 101.6 119.38 0) (unit 1)
     (in_bom yes) (on_board yes)
-    (property "Reference" "#PWR015" (id 0) (at 101.6 125.73 0)
+    (property "Reference" "#PWR024" (id 0) (at 101.6 125.73 0)
       (effects (font (size 1.27 1.27)) hide)
     )
@@
   (symbol (lib_id "arjun_symbols:CAP_CER_0u1_50V_X7R_0603") (at 111.76 106.68 0) (unit 1)
     (in_bom yes) (on_board yes)
-    (property "Reference" "C6" (id 0) (at 114.808 107.696 0)
+    (property "Reference" "C14" (id 0) (at 114.808 107.696 0)
       (effects (font (size 1.27 1.27)) (justify left))
     )
@@
   (symbol (lib_id "power:+12V") (at 175.26 101.6 0) (unit 1)
     (in_bom yes) (on_board yes)
-    (property "Reference" "#PWR017" (id 0) (at 175.26 105.41 0)
+    (property "Reference" "#PWR023" (id 0) (at 175.26 105.41 0)
       (effects (font (size 1.27 1.27)) hide)
     )
@@
   (symbol (lib_id "arjun_symbols:CAP_CER_0u1_50V_X7R_0603") (at 165.1 106.68 0) (unit 1)
     (in_bom yes) (on_board yes)
-    (property "Reference" "C7" (id 0) (at 168.148 107.696 0)
+    (property "Reference" "C15" (id 0) (at 168.148 107.696 0)
       (effects (font (size 1.27 1.27)) (justify left))
     )
@@
   (symbol (lib_id "power:GND") (at 175.26 119.38 0) (unit 1)
     (in_bom yes) (on_board yes)
-    (property "Reference" "#PWR018" (id 0) (at 175.26 125.73 0)
-      (effects (font (size 1.27 1.27)) hide)
-    )
+    (property "Reference" "#PWR025" (id 0) (at 175.26 125.73 0)
+      (effects (font (size 1.27 1.27)) hide)
+    )

Commit message: Added 8MHz Oscillator and mapped most of the MCU pins"
Parts:
- renumbered C13 to C15, C14 to C16, C15 to C17, C16 to C18
Changed lines of the file:
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@@
   (symbol (lib_id "arjun_symbols:CAP_CER_1u_25V_X5R_0603") (at 175.26 106.68 0) (unit 1)
     (in_bom yes) (on_board yes)
-    (property "Reference" "C16" (id 0) (at 178.308 107.696 0)
+    (property "Reference" "C18" (id 0) (at 178.308 107.696 0)
       (effects (font (size 1.27 1.27)) (justify left))
     )
@@
   (symbol (lib_id "arjun_symbols:CAP_CER_1u_25V_X5R_0603") (at 101.6 106.68 0) (unit 1)
     (in_bom yes) (on_board yes)
-    (property "Reference" "C13" (id 0) (at 104.648 107.696 0)
+    (property "Reference" "C15" (id 0) (at 104.648 107.696 0)
       (effects (font (size 1.27 1.27)) (justify left))
     )
@@
   (symbol (lib_id "power:GND") (at 119.38 99.06 0) (unit 1)
     (in_bom yes) (on_board yes)
-    (property "Reference" "#PWR021" (id 0) (at 119.38 105.41 0)
+    (property "Reference" "#PWR024" (id 0) (at 119.38 105.41 0)
       (effects (font (size 1.27 1.27)) hide)
     )
@@
   (symbol (lib_id "power:+3.3V") (at 101.6 101.6 0) (unit 1)
     (in_bom yes) (on_board yes)
-    (property "Reference" "#PWR022" (id 0) (at 101.6 105.41 0)
+    (property "Reference" "#PWR025" (id 0) (at 101.6 105.41 0)
       (effects (font (size 1.27 1.27)) hide)
     )
@@
   (symbol (lib_id "power:GND") (at 101.6 119.38 0) (unit 1)
     (in_bom yes) (on_board yes)
-    (property "Reference" "#PWR024" (id 0) (at 101.6 125.73 0)
+    (property "Reference" "#PWR027" (id 0) (at 101.6 125.73 0)
       (effects (font (size 1.27 1.27)) hide)
     )
@@
   (symbol (lib_id "arjun_symbols:CAP_CER_0u1_50V_X7R_0603") (at 111.76 106.68 0) (unit 1)
     (in_bom yes) (on_board yes)
-    (property "Reference" "C14" (id 0) (at 114.808 107.696 0)
+    (property "Reference" "C16" (id 0) (at 114.808 107.696 0)
       (effects (font (size 1.27 1.27)) (justify left))
     )
@@
   (symbol (lib_id "power:+12V") (at 175.26 101.6 0) (unit 1)
     (in_bom yes) (on_board yes)
-    (property "Reference" "#PWR023" (id 0) (at 175.26 105.41 0)
+    (property "Reference" "#PWR026" (id 0) (at 175.26 105.41 0)
       (effects (font (size 1.27 1.27)) hide)
     )
@@
   (symbol (lib_id "arjun_symbols:CAP_CER_0u1_50V_X7R_0603") (at 165.1 106.68 0) (unit 1)
     (in_bom yes) (on_board yes)
-    (property "Reference" "C15" (id 0) (at 168.148 107.696 0)
+    (property "Reference" "C17" (id 0) (at 168.148 107.696 0)
       (effects (font (size 1.27 1.27)) (justify left))
     )
@@
   (symbol (lib_id "power:GND") (at 175.26 119.38 0) (unit 1)
     (in_bom yes) (on_board yes)
-    (property "Reference" "#PWR025" (id 0) (at 175.26 125.73 0)
-      (effects (font (size 1.27 1.27)) hide)
-    )
+    (property "Reference" "#PWR028" (id 0) (at 175.26 125.73 0)
+      (effects (font (size 1.27 1.27)) hide)
+    )

Commit message: Added MCU pinouts for rotary encoder
Parts:
- renumbered C15 to C17, C16 to C18, C17 to C19, C18 to C20
Changed lines of the file:
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@@
   (symbol (lib_id "arjun_symbols:CAP_CER_1u_25V_X5R_0603") (at 175.26 106.68 0) (unit 1)
     (in_bom yes) (on_board yes)
-    (property "Reference" "C18" (id 0) (at 178.308 107.696 0)
+    (property "Reference" "C20" (id 0) (at 178.308 107.696 0)
       (effects (font (size 1.27 1.27)) (justify left))
     )
@@
   (symbol (lib_id "arjun_symbols:CAP_CER_1u_25V_X5R_0603") (at 101.6 106.68 0) (unit 1)
     (in_bom yes) (on_board yes)
-    (property "Reference" "C15" (id 0) (at 104.648 107.696 0)
+    (property "Reference" "C17" (id 0) (at 104.648 107.696 0)
       (effects (font (size 1.27 1.27)) (justify left))
     )
@@
   (symbol (lib_id "power:GND") (at 119.38 99.06 0) (unit 1)
     (in_bom yes) (on_board yes)
-    (property "Reference" "#PWR024" (id 0) (at 119.38 105.41 0)
+    (property "Reference" "#PWR039" (id 0) (at 119.38 105.41 0)
       (effects (font (size 1.27 1.27)) hide)
     )
@@
   (symbol (lib_id "power:+3.3V") (at 101.6 101.6 0) (unit 1)
     (in_bom yes) (on_board yes)
-    (property "Reference" "#PWR025" (id 0) (at 101.6 105.41 0)
+    (property "Reference" "#PWR037" (id 0) (at 101.6 105.41 0)
       (effects (font (size 1.27 1.27)) hide)
     )
@@
   (symbol (lib_id "power:GND") (at 101.6 119.38 0) (unit 1)
     (in_bom yes) (on_board yes)
-    (property "Reference" "#PWR027" (id 0) (at 101.6 125.73 0)
+    (property "Reference" "#PWR038" (id 0) (at 101.6 125.73 0)
       (effects (font (size 1.27 1.27)) hide)
     )
@@
   (symbol (lib_id "arjun_symbols:CAP_CER_0u1_50V_X7R_0603") (at 111.76 106.68 0) (unit 1)
     (in_bom yes) (on_board yes)
-    (property "Reference" "C16" (id 0) (at 114.808 107.696 0)
+    (property "Reference" "C18" (id 0) (at 114.808 107.696 0)
       (effects (font (size 1.27 1.27)) (justify left))
     )
@@
   (symbol (lib_id "power:+12V") (at 175.26 101.6 0) (unit 1)
     (in_bom yes) (on_board yes)
-    (property "Reference" "#PWR026" (id 0) (at 175.26 105.41 0)
+    (property "Reference" "#PWR040" (id 0) (at 175.26 105.41 0)
       (effects (font (size 1.27 1.27)) hide)
     )
@@
   (symbol (lib_id "arjun_symbols:CAP_CER_0u1_50V_X7R_0603") (at 165.1 106.68 0) (unit 1)
     (in_bom yes) (on_board yes)
-    (property "Reference" "C17" (id 0) (at 168.148 107.696 0)
+    (property "Reference" "C19" (id 0) (at 168.148 107.696 0)
       (effects (font (size 1.27 1.27)) (justify left))
     )
@@
   (symbol (lib_id "power:GND") (at 175.26 119.38 0) (unit 1)
     (in_bom yes) (on_board yes)
-    (property "Reference" "#PWR028" (id 0) (at 175.26 125.73 0)
-      (effects (font (size 1.27 1.27)) hide)
-    )
+    (property "Reference" "#PWR041" (id 0) (at 175.26 125.73 0)
+      (effects (font (size 1.27 1.27)) hide)
+    )

Commit message: Added load switch to input to limit inrush
Parts:
- removed U4: IC_LVL_MC14504BDTR2G, arjun_footprints:MC14504BDTR2G, symbol arjun_symbols:IC_LVL_MC14504BDTR2G
- added U4: IC_LVL_ONSEMI_MC14504BDTR2G, arjun_footprints:MC14504BDTR2G, symbol .arjun:IC_LVL_ONSEMI_MC14504BDTR2G
Connections:
- net +12V: now also U4.16 (VDD_OUT)
- net +3.3V: now also U4.1 (VCC_IN)
- net CLK_12V: now also U4.2 (AOUT)
- net CLK_3V3: now also U4.3 (AIN)
- net DATA_12V: now also U4.4 (BOUT)
- net DATA_3V3: now also U4.5 (BIN)
- net GND: now also U4.13 (MODE), U4.14 (FIN), U4.8 (VSS)
- net nBL_12V: now also U4.12 (EOUT)
- net nBL_3V3: now also U4.11 (EIN)
- net nLE_12V: now also U4.6 (COUT)
- net nLE_3V3: now also U4.7 (CIN)
- net nPOL_12V: now also U4.10 (DOUT)
- net nPOL_3V3: now also U4.9 (DIN)
Changed lines of the file:
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@@
     (pin "1")
-  )
-  (symbol (lib_id "arjun_symbols:IC_LVL_MC14504BDTR2G") (at 121.92 78.74 0) (unit 1)
-    (in_bom yes) (on_board yes)
-    (property "Reference" "U4" (id 0) (at 130.81 72.39 0)
-      (effects (font (size 1.524 1.524)))
-    )
-    (property "Value" "IC_LVL_MC14504BDTR2G" (id 1) (at 177.8 76.2 0)
-      (effects (font (size 1.524 1.524)) (justify left) hide)
-    )
-    (property "Footprint" "arjun_footprints:MC14504BDTR2G" (id 2) (at 177.8 78.74 0)
-      (effects (font (size 1.524 1.524)) (justify left) hide)
-    )
-    (property "Datasheet" "https://www.onsemi.com/pdf/datasheet/mc14504b-d.pdf" (id 3) (at 177.8 83.82 0)
-      (effects (font (size 1.524 1.524)) (justify left) hide)
-    )
-    (property "Manufacturer" "onsemi" (id 4) (at 177.8 87.63 0)
-      (effects (font (size 1.27 1.27)) (justify left) hide)
-    )
-    (property "ManufacturerPN" "MC14504BDTR2G" (id 5) (at 129.54 119.38 0)
-      (effects (font (size 1.27 1.27)) (justify left bottom))
-    )
-    (property "Vendor" "Digi-Key" (id 6) (at 177.8 90.17 0)
-      (effects (font (size 1.27 1.27)) (justify left) hide)
-    )
-    (property "VendorPN" "MC14504BDTR2GOSCT-ND" (id 7) (at 177.8 92.71 0)
-      (effects (font (size 1.27 1.27)) (justify left) hide)
-    )
-    (pin "1")
-    (pin "10")
-    (pin "11")
-    (pin "12")
-    (pin "13")
-    (pin "14")
-    (pin "15")
-    (pin "16")
-    (pin "2")
-    (pin "3")
-    (pin "4")
-    (pin "5")
-    (pin "6")
-    (pin "7")
-    (pin "8")
-    (pin "9")
   )
   (symbol (lib_id "power:GND") (at 101.6 119.38 0) (unit 1)
@@
     (pin "2")
   )
+  (symbol (lib_id ".arjun:IC_LVL_ONSEMI_MC14504BDTR2G") (at 121.92 78.74 0) (unit 1)
+    (in_bom yes) (on_board yes)
+    (property "Reference" "U4" (id 0) (at 130.81 72.39 0)
+      (effects (font (size 1.524 1.524)))
+    )
+    (property "Value" "IC_LVL_ONSEMI_MC14504BDTR2G" (id 1) (at 177.8 76.2 0)
+      (effects (font (size 1.524 1.524)) (justify left) hide)
+    )
+    (property "Footprint" "arjun_footprints:MC14504BDTR2G" (id 2) (at 177.8 78.74 0)
+      (effects (font (size 1.524 1.524)) (justify left) hide)
+    )
+    (property "Datasheet" "https://www.onsemi.com/pdf/datasheet/mc14504b-d.pdf" (id 3) (at 177.8 83.82 0)
+      (effects (font (size 1.524 1.524)) (justify left) hide)
+    )
+    (property "Manufacturer" "onsemi" (id 4) (at 177.8 87.63 0)
+      (effects (font (size 1.27 1.27)) (justify left) hide)
+    )
+    (property "ManufacturerPN" "MC14504BDTR2G" (id 5) (at 129.54 119.38 0)
+      (effects (font (size 1.27 1.27)) (justify left bottom))
+    )
+    (property "Vendor" "Digi-Key" (id 6) (at 177.8 90.17 0)
+      (effects (font (size 1.27 1.27)) (justify left) hide)
+    )
+    (property "VendorPN" "MC14504BDTR2GOSCT-ND" (id 7) (at 177.8 92.71 0)
+      (effects (font (size 1.27 1.27)) (justify left) hide)
+    )
+    (pin "1")
+    (pin "10")
+    (pin "11")
+    (pin "12")
+    (pin "13")
+    (pin "14")
+    (pin "15")
+    (pin "16")
+    (pin "2")
+    (pin "3")
+    (pin "4")
+    (pin "5")
+    (pin "6")
+    (pin "7")
+    (pin "8")
+    (pin "9")
+  )
   (symbol (lib_id "power:+12V") (at 175.26 101.6 0) (unit 1)

Commit message: Routing progress! Maybe 30% done.
Connections:
- net CLK_12V: now also U4.4 (BOUT); no longer U4.2 (AOUT)
- net CLK_3V3: now also U4.5 (BIN); no longer U4.3 (AIN)
- net DATA_12V: now also U4.2 (AOUT); no longer U4.4 (BOUT)
- net DATA_3V3: now also U4.3 (AIN); no longer U4.5 (BIN)
Changed lines of the file:
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@@
+		)
+	)
+	(hierarchical_label "DATA_12V"
+		(shape output)
+		(at 172.72 78.74 0)
+		(fields_autoplaced yes)
+		(effects
+			(font
+				(size 1.27 1.27)
+			)
+			(justify left)
 		)
 	)
@@
 		)
 	)
-	(hierarchical_label "DATA_12V"
-		(shape output)
-		(at 172.72 81.28 0)
+	(hierarchical_label "DATA_3V3"
+		(shape input)
+		(at 111.76 78.74 180)
 		(fields_autoplaced yes)
 		(effects
@@
 				(size 1.27 1.27)
 			)
-			(justify left)
+			(justify right)
 		)
 	)
 	(hierarchical_label "CLK_3V3"
 		(shape input)
-		(at 111.76 78.74 180)
+		(at 111.76 81.28 180)
 		(fields_autoplaced yes)
 		(effects
@@
 		(shape input)
 		(at 111.76 86.36 180)
-		(fields_autoplaced yes)
-		(effects
-			(font
-				(size 1.27 1.27)
-			)
-			(justify right)
-		)
-	)
-	(hierarchical_label "CLK_12V"
-		(shape output)
-		(at 172.72 78.74 0)
-		(fields_autoplaced yes)
-		(effects
-			(font
-				(size 1.27 1.27)
-			)
-			(justify left)
-		)
-	)
-	(hierarchical_label "DATA_3V3"
-		(shape input)
-		(at 111.76 81.28 180)
 		(fields_autoplaced yes)
 		(effects
@@
 		(fields_autoplaced yes)
 		(effects
+			(font
+				(size 1.27 1.27)
+			)
+			(justify left)
+		)
+	)
+	(hierarchical_label "CLK_12V"
+		(shape output)
+		(at 172.72 81.28 0)
+		(fields_autoplaced yes)
+		(effects
