File: pcb/STM32_Nixie.kicad_pcb (KiCad board)
At the start: 4 copper layers, 154 x 57 mm, 189 parts, among them J1 CON_SAMTEC_14P_2R_1m27_P_KEY_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, J2 CONN_USBC_RCPT_USB2.0_USB4085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, Q1 NFET_250V_10A_TPH1110FNH,L1Q, Q2 NFET_60V_0A5_2N7002KT1G, SW1 ENC_SPST_24PPR_PEC12R-4225F-S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, U1 IC_SR_MC_HV5622PG-G, U2 IC_SR_MC_HV5622PG-G, U3 IC_MCU_STM32F100C4T6B_48LQFP, U4 IC_LVL_ONSEMI_MC14504BDTR2G, U5 REG_SW_BOOST_TI_TLV61046ADBV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

Commit message: Some silk additions
Parts:
- added G***: LOGO, delo300mm_bold, B.Cu at (205.8, 105.9)
- added REF**: Symbol_HighVoltage_Triangle_6x6mm_Copper, arjun_footprints:Symbol_HighVoltage_Triangle_6x6mm_Copper, F.Cu at (224.8, 102.7)
- added REF**: Symbol_HighVoltage_Triangle_6x6mm_Copper, arjun_footprints:Symbol_HighVoltage_Triangle_6x6mm_Copper, F.Cu at (186.9, 64.9)
- added REF**: Symbol_HighVoltage_Triangle_6x6mm_Copper, arjun_footprints:Symbol_HighVoltage_Triangle_6x6mm_Copper, B.Cu at (142.9, 76.9)
- N1, N2: value Val** -> IN-3
- N3, N4, N5, N6, N7, N8: value Val** -> IN-14
- TP1: value RTC_OUT -> RTC
- TP2: value TP_KEYSTONE_5019 -> 12V
- TP3: value TP_KEYSTONE_5019 -> 3V3
- TP4: value TP_KEYSTONE_5019 -> 180V
- TP5: value TP_KEYSTONE_5019 -> VBUS
- TP6: value TP_KEYSTONE_5019 -> 5V
Other:
- board text added: "CAUTION: HIGH VOLTAGE"
- board text added: "HV ENABLED"
