File: pcb/nixie.kicad_sch (KiCad schematic)
At the start: 2 parts

Commit message: Reshuffled nixie schematic to ease with routing. Need to fix the other 3 digits next.
Parts:
- renumbered N4 to N6, R12 to R14
Changed lines of the file:
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@@
 		(on_board yes)
 		(dnp no)
-		(property "Reference" "R12"
+		(property "Reference" "R14"
 			(at 166.37 98.425 90)
 			(effects
@@
 		(instances
 			(project "STM32_Nixie"
-				(path "/962b4e87-b270-45b9-b05a-9c836fe2392e/f14ed119-44a4-4dba-a5a7-78813bb44ce1/123bc2b3-e31f-4c4e-84bd-f88f5963cf35"
-					(reference "R13")
-					(unit 1)
-				)
 				(path "/962b4e87-b270-45b9-b05a-9c836fe2392e/f14ed119-44a4-4dba-a5a7-78813bb44ce1/32b29e36-e4aa-402d-be71-eea81be37139"
 					(reference "R14")
 					(unit 1)
 				)
-				(path "/962b4e87-b270-45b9-b05a-9c836fe2392e/f14ed119-44a4-4dba-a5a7-78813bb44ce1/47fb6452-bb5d-491d-bdc1-b44524035875"
-					(reference "R11")
+				(path "/962b4e87-b270-45b9-b05a-9c836fe2392e/f14ed119-44a4-4dba-a5a7-78813bb44ce1/5f52e846-69f2-4a71-9028-f5f3e293624d"
+					(reference "R12")
 					(unit 1)
 				)
@@
 					(unit 1)
 				)
-				(path "/962b4e87-b270-45b9-b05a-9c836fe2392e/f14ed119-44a4-4dba-a5a7-78813bb44ce1/9281e11a-0024-4809-b70a-f732f328168d"
-					(reference "R12")
-					(unit 1)
-				)
 				(path "/962b4e87-b270-45b9-b05a-9c836fe2392e/f14ed119-44a4-4dba-a5a7-78813bb44ce1/d4190172-8a3a-4577-991c-8945e109fb78"
 					(reference "R15")
+					(unit 1)
+				)
+				(path "/962b4e87-b270-45b9-b05a-9c836fe2392e/f14ed119-44a4-4dba-a5a7-78813bb44ce1/db7e4f59-6b30-4946-a970-5f270ae554fe"
+					(reference "R13")
+					(unit 1)
+				)
+				(path "/962b4e87-b270-45b9-b05a-9c836fe2392e/f14ed119-44a4-4dba-a5a7-78813bb44ce1/fa830174-d583-4b93-bbb5-c9853f8c519d"
+					(reference "R11")
 					(unit 1)
 				)
@@
 		(on_board yes)
 		(dnp no)
-		(property "Reference" "N4"
+		(property "Reference" "N6"
 			(at 137.16 83.82 0)
 			(effects
@@
 		(instances
 			(project "STM32_Nixie"
-				(path "/962b4e87-b270-45b9-b05a-9c836fe2392e/f14ed119-44a4-4dba-a5a7-78813bb44ce1/123bc2b3-e31f-4c4e-84bd-f88f5963cf35"
-					(reference "N5")
-					(unit 1)
-				)
 				(path "/962b4e87-b270-45b9-b05a-9c836fe2392e/f14ed119-44a4-4dba-a5a7-78813bb44ce1/32b29e36-e4aa-402d-be71-eea81be37139"
 					(reference "N6")
 					(unit 1)
 				)
-				(path "/962b4e87-b270-45b9-b05a-9c836fe2392e/f14ed119-44a4-4dba-a5a7-78813bb44ce1/47fb6452-bb5d-491d-bdc1-b44524035875"
-					(reference "N3")
+				(path "/962b4e87-b270-45b9-b05a-9c836fe2392e/f14ed119-44a4-4dba-a5a7-78813bb44ce1/5f52e846-69f2-4a71-9028-f5f3e293624d"
+					(reference "N4")
 					(unit 1)
 				)
@@
 					(unit 1)
 				)
-				(path "/962b4e87-b270-45b9-b05a-9c836fe2392e/f14ed119-44a4-4dba-a5a7-78813bb44ce1/9281e11a-0024-4809-b70a-f732f328168d"
-					(reference "N4")
-					(unit 1)
-				)
 				(path "/962b4e87-b270-45b9-b05a-9c836fe2392e/f14ed119-44a4-4dba-a5a7-78813bb44ce1/d4190172-8a3a-4577-991c-8945e109fb78"
 					(reference "N7")
+					(unit 1)
+				)
+				(path "/962b4e87-b270-45b9-b05a-9c836fe2392e/f14ed119-44a4-4dba-a5a7-78813bb44ce1/db7e4f59-6b30-4946-a970-5f270ae554fe"
+					(reference "N5")
+					(unit 1)
+				)
+				(path "/962b4e87-b270-45b9-b05a-9c836fe2392e/f14ed119-44a4-4dba-a5a7-78813bb44ce1/fa830174-d583-4b93-bbb5-c9853f8c519d"
+					(reference "N3")
 					(unit 1)
 				)
@@
 		(on_board yes)
 		(dnp no)
-		(property "Reference" "#PWR0114"
+		(property "Reference" "#PWR034"
 			(at 180.34 97.79 0)
 			(effects
@@
 		(instances
 			(project "STM32_Nixie"
-				(path "/962b4e87-b270-45b9-b05a-9c836fe2392e/f14ed119-44a4-4dba-a5a7-78813bb44ce1/123bc2b3-e31f-4c4e-84bd-f88f5963cf35"
-					(reference "#PWR032")
-					(unit 1)
-				)
 				(path "/962b4e87-b270-45b9-b05a-9c836fe2392e/f14ed119-44a4-4dba-a5a7-78813bb44ce1/32b29e36-e4aa-402d-be71-eea81be37139"
 					(reference "#PWR034")
 					(unit 1)
 				)
-				(path "/962b4e87-b270-45b9-b05a-9c836fe2392e/f14ed119-44a4-4dba-a5a7-78813bb44ce1/47fb6452-bb5d-491d-bdc1-b44524035875"
-					(reference "#PWR033")
+				(path "/962b4e87-b270-45b9-b05a-9c836fe2392e/f14ed119-44a4-4dba-a5a7-78813bb44ce1/5f52e846-69f2-4a71-9028-f5f3e293624d"
+					(reference "#PWR037")
 					(unit 1)
 				)
@@
 					(unit 1)
 				)
-				(path "/962b4e87-b270-45b9-b05a-9c836fe2392e/f14ed119-44a4-4dba-a5a7-78813bb44ce1/9281e11a-0024-4809-b70a-f732f328168d"
-					(reference "#PWR0114")
-					(unit 1)
-				)
 				(path "/962b4e87-b270-45b9-b05a-9c836fe2392e/f14ed119-44a4-4dba-a5a7-78813bb44ce1/d4190172-8a3a-4577-991c-8945e109fb78"
 					(reference "#PWR035")
 					(unit 1)
 				)
+				(path "/962b4e87-b270-45b9-b05a-9c836fe2392e/f14ed119-44a4-4dba-a5a7-78813bb44ce1/db7e4f59-6b30-4946-a970-5f270ae554fe"
+					(reference "#PWR032")
+					(unit 1)
+				)
+				(path "/962b4e87-b270-45b9-b05a-9c836fe2392e/f14ed119-44a4-4dba-a5a7-78813bb44ce1/fa830174-d583-4b93-bbb5-c9853f8c519d"
+					(reference "#PWR033")
+					(unit 1)
+				)

Commit message: All nets routed!! (I think)
Parts:
- renumbered N6 to N7, R14 to R15
Changed lines of the file:
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@@
 		(on_board yes)
 		(dnp no)
-		(property "Reference" "R14"
+		(property "Reference" "R15"
 			(at 166.37 98.425 90)
 			(effects
@@
 		(instances
 			(project "STM32_Nixie"
-				(path "/962b4e87-b270-45b9-b05a-9c836fe2392e/f14ed119-44a4-4dba-a5a7-78813bb44ce1/32b29e36-e4aa-402d-be71-eea81be37139"
-					(reference "R14")
+				(path "/962b4e87-b270-45b9-b05a-9c836fe2392e/f14ed119-44a4-4dba-a5a7-78813bb44ce1/236b7c82-3daa-4ba4-97de-b2c4fef221cb"
+					(reference "R16")
 					(unit 1)
 				)
@@
 					(unit 1)
 				)
-				(path "/962b4e87-b270-45b9-b05a-9c836fe2392e/f14ed119-44a4-4dba-a5a7-78813bb44ce1/8d4f08ce-8f60-4112-a392-2f3cadf2f6a6"
-					(reference "R16")
+				(path "/962b4e87-b270-45b9-b05a-9c836fe2392e/f14ed119-44a4-4dba-a5a7-78813bb44ce1/7b914e47-e061-476e-92ba-d84b8eb2ac5f"
+					(reference "R14")
 					(unit 1)
 				)
@@
 		(on_board yes)
 		(dnp no)
-		(property "Reference" "N6"
+		(property "Reference" "N7"
 			(at 137.16 83.82 0)
 			(effects
@@
 		(instances
 			(project "STM32_Nixie"
-				(path "/962b4e87-b270-45b9-b05a-9c836fe2392e/f14ed119-44a4-4dba-a5a7-78813bb44ce1/32b29e36-e4aa-402d-be71-eea81be37139"
-					(reference "N6")
+				(path "/962b4e87-b270-45b9-b05a-9c836fe2392e/f14ed119-44a4-4dba-a5a7-78813bb44ce1/236b7c82-3daa-4ba4-97de-b2c4fef221cb"
+					(reference "N8")
 					(unit 1)
 				)
@@
 					(unit 1)
 				)
-				(path "/962b4e87-b270-45b9-b05a-9c836fe2392e/f14ed119-44a4-4dba-a5a7-78813bb44ce1/8d4f08ce-8f60-4112-a392-2f3cadf2f6a6"
-					(reference "N8")
+				(path "/962b4e87-b270-45b9-b05a-9c836fe2392e/f14ed119-44a4-4dba-a5a7-78813bb44ce1/7b914e47-e061-476e-92ba-d84b8eb2ac5f"
+					(reference "N6")
 					(unit 1)
 				)
@@
 		(on_board yes)
 		(dnp no)
-		(property "Reference" "#PWR034"
+		(property "Reference" "#PWR035"
 			(at 180.34 97.79 0)
 			(effects
@@
 		(instances
 			(project "STM32_Nixie"
-				(path "/962b4e87-b270-45b9-b05a-9c836fe2392e/f14ed119-44a4-4dba-a5a7-78813bb44ce1/32b29e36-e4aa-402d-be71-eea81be37139"
-					(reference "#PWR034")
+				(path "/962b4e87-b270-45b9-b05a-9c836fe2392e/f14ed119-44a4-4dba-a5a7-78813bb44ce1/236b7c82-3daa-4ba4-97de-b2c4fef221cb"
+					(reference "#PWR036")
 					(unit 1)
 				)
@@
 					(unit 1)
 				)
-				(path "/962b4e87-b270-45b9-b05a-9c836fe2392e/f14ed119-44a4-4dba-a5a7-78813bb44ce1/8d4f08ce-8f60-4112-a392-2f3cadf2f6a6"
-					(reference "#PWR036")
-					(unit 1)
-				)
+				(path "/962b4e87-b270-45b9-b05a-9c836fe2392e/f14ed119-44a4-4dba-a5a7-78813bb44ce1/7b914e47-e061-476e-92ba-d84b8eb2ac5f"
+					(reference "#PWR034")
+					(unit 1)
+				)

Commit message: Some minor tweaks and generated gerbers
Parts:
- N7: now not fitted
Changed lines of the file:
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@@
 		(in_bom yes)
 		(on_board yes)
-		(dnp no)
+		(dnp yes)
 		(property "Reference" "N7"
 			(at 137.16 83.82 0)

Commit message: Realized I got my tube naming backwards. Updated schematic with correct naming annotations
Parts:
- renumbered N7 to N8, R15 to R16
Changed lines of the file:
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@@
 		(on_board yes)
 		(dnp no)
-		(property "Reference" "R15"
+		(property "Reference" "R16"
 			(at 166.37 98.425 90)
 			(effects
@@
 		(on_board yes)
 		(dnp yes)
-		(property "Reference" "N7"
+		(property "Reference" "N8"
 			(at 137.16 83.82 0)
 			(effects
@@
 		(on_board yes)
 		(dnp no)
-		(property "Reference" "#PWR035"
+		(property "Reference" "#PWR036"
 			(at 180.34 97.79 0)
 			(effects
